File: ATmega32u4_Dev/ATmega32u4_Dev.kicad_pcb (KiCad board)
At the start: 2 copper layers, 33 parts, among them J1 USB4105-GF-A, J2 ICSP HEader 2x3, J3 Conn_01x14_Pin, J4 Conn_01x14_Pin, SW1 1825910-6, U1 ATmega32U4-A, Y1 ABM8-16.000MHZ-10-1-U-T

Commit message: changed GPIO
Parts:
- moved C8 2.22 mm to (145.5, 54.0)
- moved C9 2.22 mm to (148.8, 51.2)
- moved Y1 2.22 mm to (148.2, 53.6)
- moved C12 0.68 mm to (152.1, 57.4), turned to 180 degrees
Connections:
- net USB_DN renamed USB_N
- net USB_DP renamed USB_P
- J3 pad 1: /PB0 -> Reset
- J3 pad 10: /PC7 -> /PF4
- J3 pad 11: /PD0 -> /PF5
- J3 pad 12: /PD1 -> /PF6
- J3 pad 13: /PD2 -> MCU_5V
- J3 pad 14: /PD3 -> GND
- J3 pad 2: SCL -> /PB7
- J3 pad 3: MOSI -> MISO
- J3 pad 4: MISO -> MOSI
- J3 pad 5: /PB4 -> SCL
- J3 pad 6: /PB5 -> /PB0
- J3 pad 7: /PB6 -> /PE6
- J3 pad 8: /PB7 -> /PF0
- J3 pad 9: /PC6 -> /PF1
- J4 pad 1: GND -> /PD0
- J4 pad 10: /PF5 -> /PB5
- J4 pad 11: /PF6 -> /PB6
- J4 pad 12: /PF7 -> /PC6
- J4 pad 13: Reset -> /PC7
- J4 pad 14: MCU_5V -> /PF7
- J4 pad 2: /PD4 -> /PD1
- J4 pad 3: /PD5 -> /PD2
- J4 pad 4: /PD6 -> /PD3
- J4 pad 5: /PD7 -> /PD5
- J4 pad 6: /PE6 -> /PD4
- J4 pad 7: /PF0 -> /PD6
- J4 pad 8: /PF1 -> /PD7
- J4 pad 9: /PF4 -> /PB4
Routing:
- net MCU_5V: track 24.3 -> 79.9 mm, vias 0 -> 8
- net USB_P: track 2.69 -> 26.8 mm, vias 1 -> 2
- net USB_N: track 2.69 -> 26.7 mm, vias 1 -> 2
- net Xin: track 6.26 -> 8.79 mm
- net Xout: track 6.68 -> 8.56 mm
- net SCL: track 14.4 -> 13.6 mm
- net Reset: track 10.9 -> 10.7 mm, vias 0 -> 1

Commit message: Adjusted Layout
Parts:
- moved D2 4.80 mm to (146.7, 80.1), turned to -90 degrees
- moved C1 4.68 mm to (142.2, 83.9)
- moved FB1 4.16 mm to (144.0, 79.9), turned to 0 degrees
- moved F1 3.32 mm to (143.9, 81.9), turned to 180 degrees
- moved D3 2.60 mm to (153.7, 80.7)
- moved R7 2.60 mm to (153.2, 78.5)
- moved C2 2.17 mm to (144.8, 78.5), turned to 180 degrees
- moved D1 0.61 mm to (150.1, 79.5)
- moved J4 0.51 mm to (139.0, 51.6)
- moved R1 0.46 mm to (149.3, 82.2)
- moved R2 0.46 mm to (151.3, 82.2)
- moved J3 0.20 mm to (161.5, 51.6)
Connections:
- D1 pad 2: USB_N -> USB_P
- D1 pad 3: USB_P -> USB_N
Routing:
- net /PF6: track 0.00 -> 16.6 mm
- net /PF1: track 0.00 -> 16.4 mm
- net /PF5: track 0.00 -> 16.4 mm
- net /PF4: track 0.00 -> 16.2 mm
- net /PF0: track 0.00 -> 14.9 mm
- net /PD0: track 0.00 -> 14.1 mm
- net /PF7: track 0.00 -> 13.4 mm
- net /PD1: track 0.00 -> 12.4 mm
- net GND: track 26.0 -> 14.5 mm, vias 27 -> 26
- net /PC7: track 0.00 -> 11.3 mm
- net /PD2: track 0.00 -> 10.8 mm
- net /PE6: track 0.00 -> 9.96 mm
- net /PC6: track 0.00 -> 9.60 mm
- net /PB7: track 0.00 -> 9.58 mm
- net /PD3: track 0.00 -> 9.18 mm
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Other:
- board outline added: 25.5 x 45.2 mm

Commit message: V1
Parts:
- removed the C11 at (0.94, 0.48)
- removed the C11 at (154.9, 52.3)
- removed C2: 0.1u, Capacitor_SMD:C_0402_1005Metric
- removed D1: PRTR5V0U2X, Package_TO_SOT_SMD:SOT-143
- added C11: 0.1u, Capacitor_SMD:C_0402_1005Metric, F.Cu at (162.5, 106.0)
- added G***: LOGO, Footprints:PlaceHolder_Logo, F.Cu at (167.5, 114.2)
- added U2: USBLC6-2SC6, Package_TO_SOT_SMD:SOT-23-6, F.Cu at (158.8, 109.2)
- moved SW1 52.3 mm to (165.9, 103.9), turned to 90 degrees
- moved J2 51.1 mm to (162.0, 104.2), turned to 90 degrees
- moved R5 44.7 mm to (166.7, 99.2)
- moved C12 41.5 mm to (166.3, 96.4), turned to 90 degrees
- moved C13 38.4 mm to (159.6, 102.6), turned to -90 degrees
- moved C7 37.4 mm to (158.6, 102.6), turned to -90 degrees
- moved R3 36.2 mm to (157.2, 102.6), turned to 90 degrees
- moved R4 35.2 mm to (156.2, 102.6), turned to 90 degrees
- moved C6 34.1 mm to (154.8, 102.5), turned to -90 degrees
- moved R7 32.5 mm to (163.1, 109.5), turned to 90 degrees
- moved C3 32.2 mm to (162.4, 86.8), turned to 0 degrees
- moved U1 30.7 mm to (158.8, 94.5), turned to 90 degrees
- moved D3 30.5 mm to (165.2, 109.0), turned to 180 degrees
- moved J3 30.1 mm to (170.2, 80.5)
- moved J4 30.1 mm to (147.8, 80.5)
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Connections:
- C8 pad 1: Xin -> Xout
- C9 pad 1: Xout -> Xin
- J1 pad A6: USB_P -> Net-(J1-DP1)
- J1 pad A7: USB_N -> Net-(J1-DN1)
- J1 pad B6: USB_P -> Net-(J1-DP1)
- J1 pad B7: USB_N -> Net-(J1-DN1)
- J2 pad 1: Reset -> MCU_5V
- J2 pad 2: MISO -> SCL
- J2 pad 3: MCU_5V -> GND
- J2 pad 5: GND -> Reset
- J2 pad 6: SCL -> MISO
- J3 pad 1: Reset -> /PD7
- J3 pad 10: /PF4 -> /PB7
- J3 pad 11: /PF5 -> MISO
- J3 pad 12: /PF6 -> MOSI
- J3 pad 13: MCU_5V -> SCL
- J3 pad 14: GND -> /PB0
- J3 pad 2: /PB7 -> /PD6
- J3 pad 3: MISO -> /PD4
- J3 pad 4: MOSI -> /PD5
- J3 pad 5: SCL -> /PD3
- J3 pad 6: /PB0 -> /PD2
- J3 pad 7: /PE6 -> /PD1
- J3 pad 8: /PF0 -> /PD0
- J3 pad 9: /PF1 -> Reset
- J4 pad 1: /PD0 -> GND
- J4 pad 10: /PB5 -> /PF5
- J4 pad 11: /PB6 -> /PF4
- J4 pad 12: /PC6 -> /PF1
- J4 pad 13: /PC7 -> /PF0
- J4 pad 14: /PF7 -> /PE6
- J4 pad 2: /PD1 -> MCU_5V
- J4 pad 3: /PD2 -> /PB4
- J4 pad 4: /PD3 -> /PB5
- J4 pad 5: /PD5 -> /PB6
- J4 pad 6: /PD4 -> /PC6
- J4 pad 7: /PD6 -> /PC7
- J4 pad 8: /PD7 -> /PF7
- J4 pad 9: /PB4 -> /PF6
- Y1 pad 1: Xout -> Xin
- Y1 pad 3: Xin -> Xout
Routing:
- net MCU_5V: track 80.9 -> 109.2 mm, vias 8 -> 10
- net USB_N: track 27.6 -> 6.23 mm, vias 3 -> 1
- net USB_P: track 27.4 -> 6.23 mm, vias 3 -> 1
- net SCL: track 20.2 -> 3.15 mm, vias 1 -> 0
- net MOSI: track 18.6 -> 3.29 mm, vias 1 -> 0
- net Xout: track 8.56 -> 23.7 mm, vias 0 -> 2
- net MISO: track 16.6 -> 3.33 mm, vias 1 -> 0
- net Xin: track 8.79 -> 21.2 mm, vias 0 -> 2
- net /PB0: track 6.15 -> 16.3 mm
- net /PF6: track 16.6 -> 6.59 mm
- net /PD7: track 5.88 -> 15.5 mm
- net GND: track 14.5 -> 5.66 mm, vias 26 -> 28
- net /PF5: track 16.4 -> 7.73 mm
- net /PD6: track 5.38 -> 13.9 mm
- net /PB4: track 6.38 -> 14.7 mm
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- added copper zone on B.Cu, net GND
- added copper zone on F.Cu, net GND
Other:
- board text added: "A. Slattery 11/22/25"
- board text added: "Atmega32u4"
