File: ATmega32u4_Dev/ATmega32u4_Dev.kicad_sch (KiCad schematic)
At the start: 33 parts, among them J1 USB4105-GF-A, J2 ICSP HEader 2x3, J3 Conn_01x14_Pin, J4 Conn_01x14_Pin, SW1 1825910-6, U1 ATmega32U4-A, U2 USBLC6-2SC6, Y1 ABM8-16.000MHZ-10-1-U-T

Commit message: Adjustments to ATmega32, README files, Added SEPIC converter to voltage converters, General progress on other designs
Other:
- company: Practice -> (none)
Changed lines of the file:
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@@
 	(title_block
 		(title "ATmega32U4")
-		(company "Practice")
-		(comment 1 "Dev board PCB design")
 	)
 	(rectangle
