File: ATmega32u4_Dev 4-layer/ATmega32u4_Dev.kicad_pcb (KiCad board)
At the start: 4 copper layers, 25.5 x 38.2 mm, 34 parts, among them J1 USB4105-GF-A, J2 ICSP HEader 2x3, J3 Conn_01x14_Pin, J4 Conn_01x14_Pin, SW1 1825910-6, U1 ATmega32U4-A, U2 USBLC6-2SC6, Y1 ABM8-16.000MHZ-10-1-U-T

Commit message: Final Atmega32u4
Parts:
- SW1: footprint Inductor_SMD:L_0805_2012Metric_Pad1.05x1.20mm_HandSolder -> CustomFootPrint:Generic SW 3x4mm
- moved D1 13.7 mm to (151.2, 113.0)
- moved R8 12.7 mm to (151.7, 110.8), turned to 180 degrees
- moved SW1 3.77 mm to (166.2, 105.8), turned to -90 degrees
- moved D3 2.75 mm to (162.8, 107.9)
- moved R7 2.75 mm to (163.2, 105.7)
Routing:
- net Reset: track 24.7 -> 28.7 mm
- net /PB4: track 12.7 -> 15.7 mm
- net /PD7: track 16.1 -> 18.4 mm
- net /PB5: track 13.3 -> 15.1 mm
- net /PC7: track 26.7 -> 25.9 mm
- net /PC6: track 11.8 -> 10.9 mm, vias 1 -> 0
- net /PD6: track 15.8 -> 16.3 mm
- net GND: vias 32 -> 36
Other:
- board text added: "A. Slattery 12/08/25"
- board text removed: "A. Slattery 11/28/25"
