File: ATmega32u4_Dev 4-layer/ATmega32u4_Dev.kicad_sch (KiCad schematic)
At the start: 33 parts, among them J1 USB4105-GF-A, J2 ICSP HEader 2x3, J3 Conn_01x14_Pin, J4 Conn_01x14_Pin, SW1 1825910-6, U1 ATmega32U4-A, U2 USBLC6-2SC6, Y1 ABM8-16.000MHZ-10-1-U-T

Commit message: Final Atmega32u4
Parts:
- D2: value PTVS5V0Z1USK -> PTVS5V0Z1USKYL
- F1: value Polyfuse -> 0805L050WR
- FB1: value HI0603N300R-10 -> HI0805Q310R-10
- SW1: footprint Inductor_SMD:L_0805_2012Metric_Pad1.05x1.20mm_HandSolder -> CustomFootPrint:Generic SW 3x4mm
Changed lines of the file:
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@@
 			)
 		)
-		(property "Footprint" "Inductor_SMD:L_0805_2012Metric_Pad1.05x1.20mm_HandSolder"
+		(property "Footprint" "CustomFootPrint:Generic SW 3x4mm"
 			(at 199.39 48.26 0)
 			(effects
@@
 			)
 		)
-		(property "Value" "PTVS5V0Z1USK"
+		(property "Value" "PTVS5V0Z1USKYL"
 			(at 113.03 38.0999 90)
 			(effects
@@
 			)
 		)
-		(property "Value" "HI0603N300R-10"
+		(property "Value" "HI0805Q310R-10"
 			(at 97.7519 26.67 90)
 			(effects
@@
 			)
 		)
-		(property "Value" "Polyfuse"
+		(property "Value" "0805L050WR"
 			(at 81.28 26.67 90)
 			(effects
