File: ATiny1616_Dev/ATiny1616_Dev.kicad_sch (KiCad schematic)
At the start: 0 parts

Commit message: Some changes to attiny
Parts:
- added C1: 4.7u, symbol Device:C
- added C2, C3: 0.1u, symbol Device:C_Small
- added C4: 10u, symbol Device:C_Small
- added D1: PTVS5V0Z1USK, Diode_SMD:Nexperia_DSN1608-2_1.6x0.8mm, symbol Diode:PTVS5V0Z1USK
- added F1: Polyfuse_Small, symbol Device:Polyfuse_Small
- added FB1: FerriteBead_Small, symbol Device:FerriteBead_Small
- added J1: USB_B_Micro, symbol Connector:USB_B_Micro
- added U1: ATtiny1616-M, Package_DFN_QFN:VQFN-20-1EP_3x3mm_P0.4mm_EP1.7x1.7mm, symbol MCU_Microchip_ATtiny:ATtiny1616-M
- added U2: CH340K, Package_SO:SSOP-10-1EP_3.9x4.9mm_P1mm_EP2.1x3.3mm, symbol Interface_USB:CH340K
Connections:
- new net: C3.1, U2.10 (V3)
- new net: D1.1 (K), FB1.2
- new net: C1.2, D1.2 (A)
- new net: U1.21 (GND), U1.3 (GND)
- new net: C2.2, C4.2, U1.4 (VCC)
- new net: C1.1, F1.2, FB1.1
- new net GND: C2.1, C3.2, C4.1, U2.11 (GND), U2.3 (GND)
- new net RX: U1.1 (PA2), U2.9 (RXD)
- new net TX: U1.20 (PA1), U2.8 (TXD)
- no-connect marks 0 -> 3
