File: Voltage Conversion/Voltage Conversion.kicad_sch (KiCad schematic)
At the start: 0 parts

Commit message: Voltage Converters
Parts:
- added C1, C9: 220u, symbol Device:C
- added C10: 220u, symbol Device:C_US
- added C11, C12, C3: 10u, symbol Device:C
- added C13, C4: .1u, symbol Device:C
- added C2: 680u, symbol Device:C
- added D1: 1N5819, Diode_THT:D_DO-41_SOD81_P10.16mm_Horizontal, symbol Diode:1N5819
- added D3: B340, Diode_SMD:D_SMC, symbol Diode:B340
- added J1, J10, J11, J12, J2, J3, J4, J9: Screw_Terminal_01x01, symbol Connector:Screw_Terminal_01x01
- added L1: 33u, symbol Device:L
- added L3: 15, symbol Device:L
- added R1, R3: 1K, symbol Device:R
- added RV2, RV3: R_Potentiometer_US, symbol Device:R_Potentiometer_US
- added U2: LM2596S-ADJ, Package_TO_SOT_SMD:TO-263-5_TabPin3, symbol Regulator_Switching:LM2596S-ADJ
- added U3: TPS5431DDA, Package_SO:TI_SO-PowerPAD-8_ThermalVias, symbol Regulator_Switching:TPS5431DDA
Connections:
- new net: C1.1, C3.1, C4.1, J3.1 (Pin_1), L1.2, RV2.1
- new net: C10.1, C12.1, C13.1, J11.1 (Pin_1), L3.2, RV3.3
- new net: D1.1 (K), L1.1, U2.2 (OUT)
- new net: C9.2, D3.1 (K), L3.1, U3.8 (PH)
- new net: R1.2, RV2.3
- new net: R3.2, RV3.1
- new net: RV3.2, U3.4 (VSENSE)
- new net: C2.1, J1.1 (Pin_1), U2.1 (VIN)
- new net: C9.1, U3.1 (BOOT)
- new net: C11.1, J9.1 (Pin_1), U3.7 (VIN)
- new net: RV2.2, U2.4 (FB)
- new net GND: C1.2, C10.2, C11.2, C12.2, C13.2, C2.2, C3.2, C4.2, D1.2 (A), D3.2 (A), J10.1 (Pin_1), J12.1 (Pin_1), J2.1 (Pin_1), J4.1 (Pin_1), R1.1, R3.1, U2.3 (GND), U2.5 (~{ON}/OFF), U3.6 (GND), U3.9 (GNDPAD)
Other:
- note added: "Buck Converter"
- note added: "PWM Generation"
- note added: "Smoothing Net Work"
