File: STM32F103C8T6_Dev/STM32F103C8T6_Dev.kicad_sch (KiCad schematic)
At the start: 0 parts

Commit message: Adjustments to ATmega32, README files, Added SEPIC converter to voltage converters, General progress on other designs
Parts:
- added C1, C2: 10u, symbol Device:C_Small
- added C3: 15p, symbol Device:C_Small
- added C4, C5, C6, C7, C8, C9: 100n, symbol Device:C_Small
- added D1: PTVS5V0Z1USK, Diode_SMD:Nexperia_DSN1608-2_1.6x0.8mm, symbol Diode:PTVS5V0Z1USK
- added D2, D3: LED, symbol Device:LED
- added F1: Polyfuse_Small, symbol Device:Polyfuse_Small
- added J1: USB4105-GF-A, USB4105-GF-A:GCT_USB4105-GF-A, symbol USB4105-GF-A:USB4105-GF-A
- added R1, R2: R_Small, symbol Device:R_Small
- added U1: STM32F103CBTx, Package_QFP:LQFP-48_7x7mm_P0.5mm, symbol MCU_ST_STM32F1:STM32F103CBTx
- added U2: LT1963AxST-3.3, Package_TO_SOT_SMD:SOT-223-3_TabPin2, symbol Regulator_Linear:LT1963AxST-3.3
- added Y1: ABM8-16.000MHZ-10-1-U-T, ABM8-16.000MHZ-10-1-U-T:XTAL_ABM8-16.000MHZ-10-1-U-T, symbol ABM8-16.000MHZ-10-1-U-T:ABM8-16.000MHZ-10-1-U-T
Connections:
- new net: C1.1, D1.1 (K), F1.2, U2.1 (IN)
- new net: D2.2 (A), R1.2
- new net: D3.2 (A), R2.2
- new net: J1.A1_B12 (GND), J1.B1_A12 (GND)
- new net: J1.SH1 (SHELL_GND), J1.SH2 (SHELL_GND), J1.SH3 (SHELL_GND), J1.SH4 (SHELL_GND)
- new net +3.3V: C2.1, C4.1, C5.1, C6.1, C7.1, C8.1, R1.1, U2.3 (OUT)
- new net +5V: F1.1, J1.A4_B9 (VBUS), J1.B4_A9 (VBUS)
- new net GND: C1.2, C2.2, C3.2, C4.2, C5.2, C6.2, C7.2, C8.2, C9.2, D1.2 (A), D2.1 (K), D3.1 (K), U1.23 (VSS), U1.35 (VSS), U1.47 (VSS), U1.8 (VSSA), U2.2 (GND), Y1.2 (GND), Y1.4 (GND)
- new net XTAL_IN: C3.1, Y1.1
- new net XTAL_OUT: C9.1, Y1.3
